File: power_distro.kicad_pcb (KiCad board)
At the start: 2 copper layers, 76 x 55 mm, 37 parts, among them J1 Conn_01x02, J2 Conn_01x02, J3 Conn_01x02, J4 Conn_01x02, J5 Conn_01x02, J6 Conn_01x02, J7 Conn_01x02, J8 Conn_01x02

Commit message: Updated_mask
Other:
- board text added: "LED_Power_Distribution https://github.com/wattsy/LED_Power_distribution"
Changed lines of the file:
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@@
+		)
+	)
+	(gr_text "LED_Power_Distribution\nhttps://github.com/wattsy/LED_Power_distribution\n"
+		(at 79 91.5 270)
+		(layer "F.SilkS")
+		(effects
+			(font
+				(size 1 1)
+				(thickness 0.1)
+			)
+			(justify left bottom)
 		)
 	)
