File: power_distro.kicad_pcb (KiCad board)
At the start: 2 copper layers, 76 x 55 mm, 37 parts, among them J1 Conn_01x02, J2 Conn_01x02, J3 Conn_01x02, J4 Conn_01x02, J5 Conn_01x02, J6 Conn_01x02, J7 Conn_01x02, J8 Conn_01x02

Commit message: update for PTC
Parts:
- F1, F2, F3, F4, F5, F6, F7, F8: footprint Fuse:Fuse_Bourns_MF-RHT500 -> Fuse:Fuse_Bourns_MF-RHT1000
- moved F8 4.97 mm to (140.0, 122.5)
- moved F4 4.91 mm to (140.0, 100.4)
- moved F7 3.99 mm to (125.0, 122.5)
- moved F3 3.95 mm to (125.0, 100.3)
- moved F6 3.00 mm to (110.0, 122.5)
- moved F2 2.95 mm to (110.0, 100.3)
- moved F5 2.02 mm to (95.0, 122.5)
- moved F1 1.45 mm to (95.0, 100.3)
Routing:
- net Net-(D1-K): track 19.1 -> 20.5 mm
- net Net-(D3-K): track 20.4 -> 19.1 mm
- net Net-(D5-K): track 18.0 -> 19.1 mm
- net Net-(D4-K): track 19.6 -> 19.1 mm

Commit message: further PTC update
Parts:
- moved J_IN1 2.50 mm to (144.4, 116.8)
- moved F2 2.32 mm to (110.0, 102.6)
- moved F4 2.22 mm to (140.0, 102.6)
- moved F6 2.10 mm to (110.1, 124.6)
- moved F8 2.10 mm to (140.0, 124.6)
- moved D1 2.00 mm to (86.5, 107.5)
- moved D2 2.00 mm to (99.5, 107.5)
- moved D3 2.00 mm to (114.0, 107.5)
- moved D4 2.00 mm to (128.0, 107.5)
- moved R2 2.00 mm to (106.5, 107.5)
- moved R3 2.00 mm to (120.0, 107.5)
- moved R4 2.00 mm to (134.5, 107.5)
- moved Re1 2.00 mm to (93.0, 107.5)
- moved F5 1.90 mm to (95.1, 120.6)
- moved F7 1.90 mm to (125.0, 120.6)
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Routing:
- net Net-(D1-K): track 20.5 -> 24.4 mm
- net Net-(D4-K): track 19.1 -> 21.1 mm
- net Net-(D3-K): track 19.1 -> 21.1 mm
- net Net-(D2-K): track 19.3 -> 21.3 mm
